File: zener_vref.kicad_pcb (KiCad board)
At the start: 2 copper layers, 100 x 50 mm, 33 parts, among them J1 Conn_01x01, J2 Conn_01x01, J3 Conn_01x01, Q1 2SA733, Q2 2SC945, Q3 КТ639В, Q4 2SC945, Q5 2SC945

Commit message: Version 1.3 : 10v KC156A
Parts:
- removed C4: 22u, _сustom:LUT_CP_Radial_D5.0mm_P2.50mm
- removed the G*** at (152.0, 123.1)
- removed H5: MountingHole, MountingHole:MountingHole_2.7mm_M2.5
- removed R10: 102k, _сustom:LUT_R_L9.0mm_D3.2mm_P12.70mm_Horizontal
- removed R11, R9: 3k7, _сustom:LUT_R_L9.0mm_D3.2mm_P12.70mm_Horizontal
- removed R8: 422, _сustom:LUT_R_L9.0mm_D3.2mm_P12.70mm_Horizontal
- added C5: 470p, lut_foorprints:LUT_C_Disc_D7.5mm_W2.5mm_P5.00mm, F.Cu at (175.1, 98.4)
- added C6: 100n, lut_foorprints:LUT_C_Rect_L10.3mm_W5.0mm_P7.50mm, F.Cu at (131.9, 98.4)
- added C7: 22u, lut_foorprints:LUT_CP_Radial_D5.0mm_P2.50mm, F.Cu at (130.6, 111.1)
- added G***: LOGO, lut_foorprints:ozen_10x13, F.Cu at (104.0, 128.9)
- added Q6: S9014, lut_foorprints:LUT_TO-92, F.Cu at (170.0, 108.6)
- added RV2: 47, lut_foorprints:LUT_RPot_SP3-38B_Horizontal, F.Cu at (185.2, 117.5)
- C1: value 63n -> 22u; footprint _сustom:LUT_C_Rect_L10.3mm_W5.0mm_P7.50mm -> lut_foorprints:LUT_CP_Radial_D5.0mm_P2.50mm
- C2: value 47n -> 22u; footprint _сustom:LUT_C_Disc_D10.0mm_W2.5mm_P5.00mm -> lut_foorprints:LUT_CP_Radial_D5.0mm_P2.50mm
- C3: value u22 -> 1n; footprint _сustom:LUT_CP_Radial_D4.0mm_P2.00mm -> lut_foorprints:LUT_C_Disc_D7.5mm_W2.5mm_P5.00mm
- D1: value D -> 2v7; footprint _сustom:LUT_D_P7.62mm_Horizontal -> lut_foorprints:LUT_D_P7.62mm_Horizontal
- D2: value 1N4743A -> D; footprint _сustom:LUT_D_P10.16mm_Horizontal -> lut_foorprints:LUT_D_P7.62mm_Horizontal
- D3: value 2x КС156А -> КС156А; footprint _сustom:LUT_D_P600_R-6_P7.62mm_Vertical_AnodeUp -> lut_foorprints:LUT_D_H7.0_W9.0_P30.48_Horizontal
- J1, J2, J3: footprint _сustom:LUT_PinHeader_1x01_P2.54mm_Vertical -> lut_foorprints:LUT_Wire_Clip_2_P2.54mm
- Q1: value 2SA733 -> KT639; footprint _сustom:LUT_TO-92 -> lut_foorprints:LUT_TO-126-3_Vertical
- Q2, Q4, Q5: value 2SC945 -> S9015; footprint _сustom:LUT_TO-92 -> lut_foorprints:LUT_TO-92
- Q3: value КТ639В -> S9014; footprint _сustom:LUT_TO-126-3_Vertical -> lut_foorprints:LUT_TO-92
- R1: value 32k -> 6k8; footprint _сustom:LUT_R_L9.0mm_D3.2mm_P12.70mm_Horizontal -> lut_foorprints:LUT_R_L9.9mm_D3.6mm_P12.70mm_Horizontal
- R2: value 470 -> 6k8; footprint _сustom:LUT_R_L9.0mm_D3.2mm_P12.70mm_Horizontal -> lut_foorprints:LUT_R_L9.9mm_D3.6mm_P12.70mm_Horizontal
- R3: value 150k -> trim; footprint _сustom:LUT_R_L9.0mm_D3.2mm_P12.70mm_Horizontal -> lut_foorprints:LUT_R_L9.9mm_D3.6mm_P12.70mm_Horizontal
- R4: value 825 -> 1k8; footprint _сustom:LUT_R_L9.0mm_D3.2mm_P12.70mm_Horizontal -> lut_foorprints:LUT_R_L9.9mm_D3.6mm_P12.70mm_Horizontal
- R5: value 20k -> 50k; footprint _сustom:LUT_R_L9.0mm_D3.2mm_P12.70mm_Horizontal -> lut_foorprints:LUT_R_L9.9mm_D3.6mm_P12.70mm_Horizontal
- R6: value 20k -> 3k7; footprint _сustom:LUT_R_L9.0mm_D3.2mm_P12.70mm_Horizontal -> lut_foorprints:LUT_R_L9.9mm_D3.6mm_P12.70mm_Horizontal
- R7: value 590 -> 4k7; footprint _сustom:LUT_R_L9.0mm_D3.2mm_P12.70mm_Horizontal -> lut_foorprints:LUT_R_L9.9mm_D3.6mm_P12.70mm_Horizontal
- RV1: footprint _сustom:LUT_RPot_SP3-38B_Horizontal -> lut_foorprints:LUT_RPot_SP3-38B_Horizontal
- moved H4 101.2 mm to (93.8, 132.7)
- moved H3 100.3 mm to (185.2, 132.7)
- moved Q1 72.9 mm to (104.0, 108.6), turned to 90 degrees
- moved C2 58.0 mm to (123.0, 121.3), turned to 270 degrees
- moved J2 56.0 mm to (125.6, 130.8), turned to 180 degrees
- moved C1 48.8 mm to (112.9, 128.3), turned to 270 degrees
- moved H2 42.2 mm to (185.2, 90.8)
- moved H1 42.2 mm to (93.8, 90.8)
- moved J3 41.9 mm to (120.5, 98.4)
- moved C3 35.6 mm to (153.5, 103.5), turned to 90 degrees
- moved R5 28.2 mm to (163.7, 118.1)
- moved D1 26.3 mm to (117.9, 123.2)
- moved R2 25.4 mm to (114.1, 116.2), turned to 0 degrees
- moved J1 25.3 mm to (120.5, 106.0), turned to 180 degrees
- moved Q2 24.3 mm to (148.4, 103.5), turned to 90 degrees
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Connections:
- C1 pad 1: VDC -> Net-(C1-Pad1)
- C2 pad 1: V+15 -> Net-(C2-Pad1)
- C3 pad 1: V+15 -> Net-(C3-Pad1)
- C3 pad 2: GND -> V+10.00
- D1 pad 1: V+15 -> Net-(C2-Pad1)
- D1 pad 2: Net-(D1-Pad2) -> GND
- D2 pad 2: GND -> Net-(C2-Pad1)
- D3 pad 1: Net-(D3-Pad1) -> Net-(D2-Pad1)
- J1 pad 1: VDC -> +VSW
- J2 pad 1: V+15 -> GND
- J3 pad 1: GND -> V+10.00
- Q1 pad 1: Net-(Q1-Pad1) -> +VSW
- Q1 pad 2: Net-(Q1-Pad2) -> V+10.00
- Q2 pad 1: Net-(D1-Pad2) -> Net-(Q1-Pad3)
- Q2 pad 2: Net-(Q2-Pad2) -> Net-(C3-Pad1)
- Q2 pad 3: Net-(D2-Pad1) -> V+10.00
- Q3 pad 1: VDC -> Net-(Q3-Pad1)
- Q3 pad 2: V+15 -> Net-(D2-Pad1)
- Q3 pad 3: Net-(Q1-Pad1) -> Net-(C3-Pad1)
- Q4 pad 1: Net-(Q4-Pad1) -> +VSW
- Q4 pad 3: Net-(Q4-Pad3) -> Net-(C3-Pad1)
- Q5 pad 1: Net-(Q4-Pad1) -> +VSW
- Q5 pad 2: Net-(Q1-Pad3) -> Net-(Q4-Pad2)
- Q5 pad 3: Net-(D3-Pad1) -> Net-(Q4-Pad2)
- R1 pad 1: VDC -> +VSW
- R1 pad 2: Net-(D2-Pad1) -> Net-(C1-Pad1)
- R2 pad 1: VDC -> Net-(C1-Pad1)
- R2 pad 2: Net-(Q2-Pad2) -> Net-(C2-Pad1)
- R3 pad 1: Net-(D1-Pad2) -> V+10.00
- R3 pad 2: GND -> Net-(R3-Pad2)
- R4 pad 1: V+15 -> V+10.00
- R4 pad 2: Net-(R4-Pad2) -> Net-(R3-Pad2)
- R5 pad 1: VDC -> Net-(Q3-Pad1)
- R5 pad 2: Net-(Q4-Pad2) -> GND
- R6 pad 1: VDC -> V+10.00
- R6 pad 2: Net-(Q1-Pad3) -> Net-(R6-Pad2)
- R7 pad 1: V+15 -> Net-(R7-Pad1)
- R7 pad 2: Net-(D3-Pad1) -> GND
- RV1 pad 1: Net-(R9-Pad1) -> Net-(D2-Pad1)
- RV1 pad 2: Net-(Q4-Pad3) -> Net-(D2-Pad1)
- RV1 pad 3: Net-(R8-Pad2) -> Net-(R3-Pad2)
Routing:
- net (no net): track 342.9 -> 0.00 mm
- net GND: track 139.0 -> 5.08 mm
- net +VSW: track 0.00 -> 92.7 mm, vias 0 -> 3
- net V+10.00: track 0.00 -> 91.1 mm
- net V+15: track 75.9 -> 0.00 mm
- net VDC: track 73.0 -> 0.00 mm
- net Net-(D2-Pad1): track 12.1 -> 52.0 mm
- net Net-(C3-Pad1): track 0.00 -> 27.8 mm
- net Net-(C5-Pad2): track 0.00 -> 27.0 mm
- net Net-(Q1-Pad3): track 19.4 -> 46.0 mm
- net Net-(Q4-Pad2): track 7.87 -> 32.7 mm
- net Net-(D3-Pad1): track 21.7 -> 0.00 mm
- net Net-(R7-Pad1): track 0.00 -> 19.3 mm
- net Net-(Q4-Pad1): track 18.4 -> 0.00 mm
- net Net-(C1-Pad1): track 0.00 -> 17.7 mm
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- added copper zone on B.Cu, net GND
- added copper zone on B.Cu, net V+10.00
Other:
- board text added: "10V"
- board text added: "10V trim"
- board text added: "Input : 13-40V Output : 10V Max. load : 25mA"
- board text added: "Vin"
- board text added: "https://github.com/2BatBox/zener_vref Zener voltage reference. Rev 1.3"
- board text added: "zen. cur. trim"
- board text removed: "+15V"
- board text removed: "+15V trim"
- board text removed: "Input voltage range: 16-45V Output voltage: 15V Max. load current : 20mA Zener: 2x КС156А (5.6V 6.3mA) ---------------------- https://github.com/2SilentJay/zener_vref"
- board text removed: "V+"
- board text removed: "Zener voltage reference. Rev 1.2 ----------------------"
